Commit message: Updated sick_lms1xx_mount.urdf.xacro: added min_range to macro.

File: jackal_description/urdf/accessories/sick_lms1xx_mount.urdf.xacro (robot description, xacro)
@@ -27,6 +27,10 @@
 <robot xmlns:xacro="http://www.ros.org/wiki/xacro">
   <xacro:include filename="$(find lms1xx)/urdf/sick_lms1xx.urdf.xacro" />
-  <xacro:macro name="sick_lms1xx_mount" params="prefix topic parent_link *origin">
-    <xacro:sick_lms1xx frame="${prefix}_laser" topic="${topic}" />
+  <xacro:macro name="sick_lms1xx_mount" params="prefix topic parent_link min_range max_range *origin">
+    <!--xacro:sick_lms1xx frame="${prefix}_laser" topic="${topic}" /-->
+    <xacro:sick_lms1xx frame="${prefix}_laser"
+                        topic="${topic}"
+                        min_range="${min_range}"
+                        max_range="${max_range}"/>
     <joint name="${prefix}_laser_mount_joint" type="fixed">
       <xacro:insert_block name="origin" />
