Commit message: Updated jackal.urdf.xacro: increased mass to prevent roll over because of the arm.

File: jackal_description/urdf/jackal.urdf.xacro (robot description, xacro)
@@ -103,5 +103,5 @@
       <!-- Center of mass -->
       <origin xyz="0.012  0.002 0.067" rpy="0 0 0"/>
-      <mass value="16.523"/>
+      <mass value="160.523"/> <!-- Default: 16.523 -->
       <!-- Moments of inertia: ( chassis without wheels ) -->
       <inertia
@@ -119,4 +119,10 @@
         <material name="yellow" />
       </visual>
+      <collision>
+        <!--origin xyz="0 0 0" rpy="0 0 0"/-->
+        <geometry>
+          <mesh filename="package://jackal_description/meshes/jackal-fender.stl"/>
+        </geometry>
+      </collision>
     </link>
   </xacro:unless>
@@ -129,4 +135,10 @@
         <material name="yellow" />
       </visual>
+      <collision>
+        <!--origin xyz="0 0 0" rpy="0 0 0"/-->
+        <geometry>
+          <mesh filename="package://jackal_description/meshes/accessory_fender.stl"/>
+        </geometry>
+      </collision>
     </link>
     <link name="front_fender_accessory_link"/>
@@ -150,4 +162,10 @@
         <material name="yellow" />
       </visual>
+      <collision>
+        <!--origin xyz="0 0 0" rpy="0 0 0"/-->
+        <geometry>
+          <mesh filename="package://jackal_description/meshes/jackal-fender.stl"/>
+        </geometry>
+      </collision>
     </link>
   </xacro:unless>
@@ -160,4 +178,10 @@
         <material name="yellow" />
       </visual>
+      <collision>
+        <!--origin xyz="0 0 0" rpy="0 0 0"/-->
+        <geometry>
+          <mesh filename="package://jackal_description/meshes/accessory_fender.stl"/>
+        </geometry>
+      </collision>
     </link>
     <link name="rear_fender_accessory_link"/>
@@ -197,4 +221,10 @@
       <material name="black" />
     </visual>
+    <collision>
+      <geometry>
+        <cylinder radius="0.026" length="0.016" />
+      </geometry>
+      <origin xyz="0 0 0.008" />
+    </collision>
   </link>
   <joint name="navsat_joint" type="fixed">

Commit message: Updated jackal.urdf.xacro: updated chassis_link mass back to its original value.

File: jackal_description/urdf/jackal.urdf.xacro (robot description, xacro)
@@ -103,5 +103,5 @@
       <!-- Center of mass -->
       <origin xyz="0.012  0.002 0.067" rpy="0 0 0"/>
-      <mass value="160.523"/> <!-- Default: 16.523 -->
+      <mass value="16.523"/> <!-- Default: 16.523 -->
       <!-- Moments of inertia: ( chassis without wheels ) -->
       <inertia
